File: A500+ 2MB.brd (EAGLE design)
At the start: 81.3 x 27.9 mm, 50 parts, among them U1 1Mx16 DRAM, U2 74AHC1G08DBV

Commit message: Latest version
Parts:
- moved !RAS0 3.81 mm to (67.3, 17.8)
- moved DRA9 3.81 mm to (73.7, 8.89)
- moved DRD1 3.81 mm to (67.3, 22.9)
- moved DRD3 3.81 mm to (67.3, 25.4)
- moved PAD3 3.81 mm to (67.3, 5.08)
- moved R1 3.81 mm to (73.7, 14.0)
- moved VCC@3 3.81 mm to (67.3, 2.54)
- moved DRD0 3.81 mm to (74.9, 20.3)
- moved DRD2 3.81 mm to (74.9, 22.9)
- moved GND@4 3.81 mm to (74.9, 25.4)
- moved C4 2.54 mm to (68.6, 9.02)
- moved R2 2.54 mm to (64.8, 11.4)
- moved U2 2.54 mm to (68.6, 12.7)
- moved !CASL 2.54 mm to (61.0, 17.8)
- moved !RAS1 2.54 mm to (53.3, 17.8)
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Routing:
- net +5V: track 73.5 -> 70.9 mm
- net DRD13: track 31.7 -> 29.1 mm
- net DRD12: track 24.3 -> 21.7 mm
- net DRD14: track 27.8 -> 25.3 mm
- net DRD15: track 35.2 -> 32.7 mm
- net !CASU: track 32.5 -> 30.3 mm
- net DRD9: track 26.3 -> 24.3 mm
- net DRD11: track 29.7 -> 27.7 mm
- net !DWE: track 31.9 -> 29.9 mm
- net DRD10: track 27.4 -> 25.8 mm
- net DRA9: track 42.5 -> 41.2 mm
- net DRD3: track 50.1 -> 48.8 mm
- net DRD1: track 49.8 -> 48.6 mm
- net DRD0: track 49.5 -> 48.3 mm
- net DRD2: track 53.3 -> 52.1 mm
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Other:
- board size 81.3 x 27.9 mm -> 77.5 x 27.9 mm
